Commit message: Add files via upload

File: clhero_description/robots/clhero.robot.xacro (robot description, xacro)
@@ -10,4 +10,5 @@
 <xacro:include filename="$(find clhero_description)/urdf/sensores/imu.xacro"/>
 <xacro:include filename="$(find clhero_description)/urdf/sensores/hokuyo_sensor.xacro"/>
+<xacro:include filename="$(find realsense2_description)/urdf/_d435.urdf.xacro"/>
 <!-- Declaracion del plugin gazebo_ros_control -->
 <gazebo>
@@ -67,3 +68,6 @@
     <origin xyz="${300/1000} 0 0" rpy="0 0 0"/>
 </hokuyo_sensor-->
+<sensor_d435 parent="base_link">
+    <origin xyz="0.27 0 -0.01" rpy="0 0 0"/>
+</sensor_d435>
 </robot>

File: clhero_description/robots/clhero.urdf.xacro (robot description, xacro)
@@ -10,4 +10,5 @@
 <xacro:include filename="$(find clhero_description)/urdf/sensores/imu.xacro"/>
 <xacro:include filename="$(find clhero_description)/urdf/sensores/hokuyo_sensor.xacro"/-->
+<xacro:include filename="$(find realsense2_description)/urdf/_d435.urdf.xacro"/>
 <!-- Declaracion del plugin gazebo_ros_control -->
 <gazebo>
@@ -46,3 +47,6 @@
     <origin xyz="${300/1000} 0 0" rpy="0 0 0"/>
 </hokuyo_sensor-->
+<sensor_d435 parent="base_link">
+    <origin xyz="0.27 0 -0.01" rpy="0 0 0"/>
+</sensor_d435>
 </robot>
