Commit message: Add files via upload

File: clhero_description/robots/clhero.urdf.xacro (robot description, xacro)
@@ -8,6 +8,6 @@
 <xacro:include filename="$(find clhero_description)/urdf/base.xacro"/>
 <!--xacro:include filename="$(find clhero_description)/urdf/sensores/kinect_camera.xacro"/>
-<xacro:include filename="$(find clhero_description)/urdf/sensores/imu.xacro"/>
-<xacro:include filename="$(find clhero_description)/urdf/sensores/hokuyo_sensor.xacro"/-->
+<xacro:include filename="$(find clhero_description)/urdf/sensores/imu.xacro"/-->
+<xacro:include filename="$(find clhero_description)/urdf/sensores/hokuyo_sensor.xacro"/>
 <xacro:include filename="$(find realsense2_description)/urdf/_d435.urdf.xacro"/>
 <!-- Declaracion del plugin gazebo_ros_control -->
@@ -41,10 +41,10 @@
 </kinect_camera-->
 <!-- Instanciacion de la IMU dentro de la descripcion del robot -->
-<!--imu name="imu1" parent_link="base_link">
-    <origin xyz="${0/1000} ${0/1000} ${40/1000}" rpy="0 0 ${pi/2}"/>
-</imu-->
-<!--hokuyo_sensor sensor_name="hokuyo" parent_name="base_link">
-    <origin xyz="${300/1000} 0 0" rpy="0 0 ${pi/2}"/>
-</hokuyo_sensor-->
+<imu name="base_imu_link" parent_link="base_link">
+    <origin xyz="${0/1000} ${0/1000} ${40/1000}" rpy="0 0 0"/>
+</imu>
+<hokuyo_sensor sensor_name="hokuyo" parent_name="base_link">
+    <origin xyz="-0.26 0 ${40/1000}" rpy="0 0 ${pi}"/>
+</hokuyo_sensor>
 <sensor_d435 parent="base_link">
     <origin xyz="-0.27 0 -0.01" rpy="0 0 ${pi}"/>

File: clhero_description/urdf/sensores/hokuyo_sensor.xacro (robot description, xacro)
@@ -2,5 +2,5 @@
 <robot name="hokuyo_sensor" xmlns:xacro="http://ros.org/wiki/xacro">
     <xacro:macro name="hokuyo_sensor" params="sensor_name parent_name *origin">
-        <link name="${sensor_name}_hokuyo_base">
+        <link name="laser">
             <inertial>
                 <mass value="0.1"/>
@@ -23,8 +23,8 @@
             <xacro:insert_block name="origin"/>
             <parent link="${parent_name}"/>
-            <child link="${sensor_name}_hokuyo_base"/>
+            <child link="laser"/>
         </joint>
         <!-- hokuyo -->
-        <gazebo reference="${sensor_name}_hokuyo_base">
+        <gazebo reference="laser">
           <material>Gazebo/blue</material>
           <sensor type="ray" name="head_hokuyo_sensor">
@@ -58,5 +58,5 @@
             <plugin name="gazebo_ros_head_hokuyo_controller" filename="libgazebo_ros_laser.so">
               <topicName>/robotest/laser/scan</topicName>
-              <frameName>${sensor_name}_hokuyo_base</frameName>
+              <frameName>laser</frameName>
             </plugin>
           </sensor>
