Commit message: realsense included in urdf

File: clhero_description/urdf/base.xacro (robot description, xacro)
@@ -49,5 +49,6 @@
     <parent link="base_footprint"/>
     <child link="base_link"/>
-    <origin xyz="0 0 ${w_radius*2}" rpy="0 0 0"/>
+    <!--origin xyz="0 0 ${w_radius*2}" rpy="0 0 0"/-->
+    <origin xyz="0 0 ${0.04}" rpy="0 0 ${pi}"/>
 </joint>
 </robot>
